File: Macrotype-0/Macrotype-0.kicad_pcb (KiCad board)
At the start: 2 copper layers, 30 parts, among them U1 ProMicro

Commit message: Update 1.1
Connections:
- D1 pad 1: ROW0 -> ROW1
- D2 pad 1: ROW1 -> ROW0
- D3 pad 1: ROW0 -> ROW1
- D4 pad 1: ROW1 -> ROW0
- MX1 pad 1: unconnected-(MX1-Pad1) -> COL2
- MX11 pad 1: COL1 -> COL2
- MX4 pad 1: COL1 -> COL0
- MX6 pad 1: COL1 -> COL2
- MX9 pad 1: unconnected-(MX9-Pad1) -> COL0
Routing:
- net COL1: track 0.00 -> 97.4 mm
- net ROW3: track 0.00 -> 77.6 mm
- net ROW1: track 0.00 -> 77.6 mm
- net COL0: track 0.00 -> 77.3 mm
- net GND: track 0.00 -> 39.4 mm
- net COL2: track 0.00 -> 39.2 mm
- net ROW5: track 0.00 -> 38.8 mm
- net ROW0: track 0.00 -> 38.8 mm
- net ROW4: track 0.00 -> 38.8 mm
- net ROW2: track 0.00 -> 38.8 mm
- net Net-(U1-RST): track 0.00 -> 33.0 mm
- net Net-(D4-A): track 0.00 -> 8.68 mm
- net Net-(D9-A): track 0.00 -> 8.68 mm
- net Net-(D14-A): track 0.00 -> 8.68 mm
- net Net-(D5-A): track 0.00 -> 8.68 mm
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
Commit message: Update 1.2
Parts:
- moved U1 0.30 mm to (76.5, 74.6)
Connections:
- U1 pad 1: unconnected-(U1-D3-TX-Pad1) -> COL0
- U1 pad 10: unconnected-(U1-E6-Pad10) -> ROW3
- U1 pad 11: unconnected-(U1-B4-Pad11) -> ROW4
- U1 pad 12: unconnected-(U1-B5-Pad12) -> ROW5
- U1 pad 5: unconnected-(U1-D1-Pad5) -> ROW0
- U1 pad 6: unconnected-(U1-D0-Pad6) -> ROW1
- U1 pad 7: unconnected-(U1-D4-Pad7) -> COL2
- U1 pad 8: unconnected-(U1-C6-Pad8) -> COL1
- U1 pad 9: unconnected-(U1-D7-Pad9) -> ROW2
Routing:
- net COL2: track 39.2 -> 127.7 mm
- net ROW5: track 38.8 -> 103.6 mm
- net COL1: track 97.4 -> 147.1 mm
- net ROW4: track 38.8 -> 84.5 mm
- net ROW2: track 38.8 -> 78.7 mm
- net ROW0: track 38.8 -> 75.8 mm
- net ROW3: track 77.6 -> 98.1 mm
- net ROW1: track 77.6 -> 95.7 mm
- net COL0: track 77.3 -> 87.2 mm
Other:
- board outline added: 116.5 x 58 mm
